File: Schematics/EPS/Flight Model/PQ60 EPS FV2.sch (EAGLE design)
At the start: 28 parts, among them U1 LTC3105EDDPBF, U2 LTC3105EDDPBF, U3 LTC3105EDDPBF, U4 LTC4413EDDPBF, U5 LTC4413EDDPBF, U6 TPS63001DRCR, X1-BOT FX8C-60S-SV, X1-TOP FX8C-60P-SV

Commit message: EPS.brd
Parts:
- removed X1-BOT: FX8C-60S-SV, PQ60:FX8C-60S-SV
- removed X1-TOP: FX8C-60P-SV, PQ60:FX8C-60P-SV
- added C11, C12, C13: 4.7uF, adafruit:C-USC0805
- added C14, C15, C16: 1uF, adafruit:C-USC0805
- added R10, R12, R13: 4.7k, adafruit:R-US_R0805
- added R11, R14, R9: 15k, adafruit:R-US_R0805
- added R3, R4, R5, R6: 35.7k, adafruit:R-US_R0805
- added R7, R8: 10k, adafruit:R-US_R0805
- added SJ1, SJ2, SLAVE_GND, SLAVE_SCL, SLAVE_SDA, SLAVE_VS: (no value), jumper:SJ
- added U$2: FX8C-060S-SV(92), PQ60:FX8C-060S-SV(92)
- added U$3: FX8C-060P-SV(92), PQ60:FX8C-060P-SV(92)
- added U10: INA3221AIRGVT, INA3221:INA3221AIRGVT
- added U7, U8: TPS2552DBVT, TPS2552:TPS2552DBVT
- BATTERY, SWITCH: value (none) -> 332-02; device pinhead:PINHD-1X2 -> con-garry:332-02
Connections:
- removed net +3V3_SW[1]: X1-BOT.+3.3V_SW1, X1-TOP.+3.3V_SW1
- removed net +3V3_SW[2]: X1-BOT.+3.3V_SW2, X1-TOP.+3.3V_SW2
- removed net +3V3_SW[3]: X1-BOT.+3.3V_SW3, X1-TOP.+3.3V_SW3
- removed net GPIO[10]: X1-BOT.GPIO10, X1-TOP.GPIO10
- removed net GPIO[11]: X1-BOT.GPIO11, X1-TOP.GPIO11
- removed net GPIO[12]: X1-BOT.GPIO12, X1-TOP.GPIO12
- removed net GPIO[13]: X1-BOT.GPIO13, X1-TOP.GPIO13
- removed net GPIO[14]: X1-BOT.GPIO14, X1-TOP.GPIO14
- removed net GPIO[1]: X1-BOT.GPIO1, X1-TOP.GPIO1
- removed net GPIO[2]: X1-BOT.GPIO2, X1-TOP.GPIO2
- removed net GPIO[3]: X1-BOT.GPIO3, X1-TOP.GPIO3
- removed net GPIO[4]: X1-BOT.GPIO4, X1-TOP.GPIO4
- removed net GPIO[5]: X1-BOT.GPIO5, X1-TOP.GPIO5
- removed net GPIO[6]: X1-BOT.GPIO6, X1-TOP.GPIO6
- removed net GPIO[7]: X1-BOT.GPIO7, X1-TOP.GPIO7
- removed net GPIO[8]: X1-BOT.GPIO8, X1-TOP.GPIO8
- removed net GPIO[9]: X1-BOT.GPIO9, X1-TOP.GPIO9
- removed net NC@34: X1-BOT.NC@1, X1-TOP.NC@1
- removed net NC@35: X1-BOT.NC@2, X1-TOP.NC@2
- removed net NC@36: X1-BOT.NC@3, X1-TOP.NC@3
- removed net NC@42: X1-BOT.NC@5, X1-TOP.NC@5
- removed net NC@43: X1-BOT.NC@6, X1-TOP.NC@6
- removed net NC@56: X1-BOT.NC@7, X1-TOP.NC@7
- removed net SPI_CS: X1-BOT.SS, X1-TOP.SS
- removed net SPI_MISO: X1-BOT.MISO, X1-TOP.MISO
- removed net SPI_MOSI: X1-BOT.MOSI, X1-TOP.MOSI
- removed net SPI_SCK: X1-BOT.SCK, X1-TOP.SCK
- removed net USB_N: X1-BOT.USB_N, X1-TOP.USB_N
- removed net USB_P: X1-BOT.USB_P, X1-TOP.USB_P
- removed net VBUS: C8.2, C9.2, R1.2, R2.2, SWITCH.2, U5.OUTA, U5.OUTB, U6.EN, U6.PS/SYNC, U6.VIN, U6.VINA, X1-BOT.VBUS@1, X1-BOT.VBUS@2, X1-BOT.VBUS@3, X1-TOP.VBUS@1, X1-TOP.VBUS@2, X1-TOP.VBUS@3
- removed net VBUS_SW[1]: X1-BOT.VBUS_SW1, X1-TOP.VBUS_SW1
- removed net VBUS_SW[2]: X1-BOT.VBUS_SW2, X1-TOP.VBUS_SW2
- removed net VBUS_SW[3]: X1-BOT.VBUS_SW3, X1-TOP.VBUS_SW3
- new net $N70: BATTERY-1.S, C8.2, SWITCH-1.S, U5.OUTA, U5.OUTB
- new net +3V3_SW1: U$2.+3V3_SW1@1, U$2.+3V3_SW1@2
- new net +3V3_SW2: U$2.+3V3_SW2@1, U$2.+3V3_SW2@2
- new net +3V3_SW3: U$2.+3V3_SW3@1, U$2.+3V3_SW3@2
- new net BATTERY: C9.2, R5.1, U6.EN, U6.PS/SYNC, U6.VIN, U6.VINA, U7.IN
- new net BATV: R1.2, R2.2, U$2.BATV@1, U$2.BATV@2, U$2.BATV@3, U$2.BATV@4, U7.OUT
- new net BATV_SW1: U$2.BATV_SW1@1, U$2.BATV_SW1@2
- new net BATV_SW2: U$2.BATV_SW2@1, U$2.BATV_SW2@2
- new net BATV_SW3: U$2.BATV_SW3@1, U$2.BATV_SW3@2
- new net GPIO0: U$2.GPIO0
- new net GPIO1: U$2.GPIO1
- new net GPIO10: U$2.GPIO10, U$3.GPIO10
- new net GPIO11: U$2.GPIO11, U$3.GPIO11
- new net GPIO12: U$2.GPIO12, U$3.GPIO12
- new net GPIO2: U$2./SS/GPIO2, U$3./SS/GPIO2
- new net GPIO3: U$2.GPIO3, U$3.GPIO3
- new net GPIO4: U$2.GPIO4, U$3.GPIO4
- new net GPIO5: U$2.GPIO5, U$3.GPIO5
- new net GPIO6: U$2.GPIO6, U$3.GPIO6
- new net GPIO7: U$2.GPIO7, U$3.GPIO7
- new net GPIO8: U$2.GPIO8, U$3.GPIO8
- new net GPIO9: U$2.GPIO9, U$3.GPIO9
- new net MISO: U$2.MISO, U$3.MISO
- new net MOSI: U$2.MOSI, U$3.MOSI
- new net N$13: R3.1, U7.ILIM
- new net N$14: R5.2, U7.~FAULT
- new net N$15: R6.2, U8.~FAULT
- new net N$16: SJ1.2, U8.EN
- new net N$17: SJ2.2, U7.EN
- new net N$18: SLAVE_GND.2, SLAVE_SCL.2, SLAVE_SDA.2, SLAVE_VS.2, U10.A0
- new net N$19: C11.1, U1.LDO
- new net N$20: C12.1, U2.LDO
- new net N$21: C13.1, U3.LDO
- new net N$22: C14.1, U2.AUX
- new net N$23: C15.1, U3.AUX
- new net N$24: C16.1, U1.AUX
- new net N$25: R10.2, R9.1, U2.FB
- new net N$26: R13.2, R14.1, U3.FB
- new net N$27: R11.1, R12.2, U1.FB
- new net SCK: U$2.SCK, U$3.SCK
- new net SCL: U$2.SCL
- new net SDA: U$2.SDA
- new net UNPROTECTED3V3: C10.2, R6.1, U6.FB, U6.VOUT, U8.IN
- new net VIN1+: U10.IN+1
- new net VIN1-: U10.IN-1
- new net VIN2+: U10.IN+2
- new net VIN2-: U10.IN-2
- new net VIN3+: U10.IN+3
- new net VIN3-: U10.IN-3
- net !RST: now also U$2./RST; no longer X1-BOT.RST, X1-TOP.RST
- net +3V3: now also R7.1, R8.1, SLAVE_VS.1, U$2.+3V3@1, U$2.+3V3@2, U$2.+3V3@3, U$2.+3V3@4, U10.VS, U8.OUT; no longer C10.2, U6.FB, U6.VOUT, X1-BOT.+3.3V@1, X1-BOT.+3.3V@2, X1-BOT.+3.3V@3, X1-TOP.+3.3V@1, X1-TOP.+3.3V@2, X1-TOP.+3.3V@3
- net GND: now also BATTERY-2.S, C11.2, C12.2, C13.2, C14.2, C15.2, C16.2, R10.1, R12.1, R13.1, R3.2, R4.2, SJ1.1, SJ2.1, SLAVE_GND.1, U$2.GND, U$2.RTN_+3V3@1, U$2.RTN_+3V3@2, U$2.RTN_+3V3@3, U$2.RTN_+3V3@4, U$2.RTN_+3V3_SW1@1, U$2.RTN_+3V3_SW1@2, U$2.RTN_+3V3_SW2@1, U$2.RTN_+3V3_SW2@2, U$2.RTN_+3V3_SW3@1, U$2.RTN_+3V3_SW3@2, U$2.RTN_BATV@1, U$2.RTN_BATV@2, U$2.RTN_BATV@3, U$2.RTN_BATV@4, U$2.RTN_BATV_SW1@1, U$2.RTN_BATV_SW1@2, U$2.RTN_BATV_SW2@1, U$2.RTN_BATV_SW2@2, U$2.RTN_BATV_SW3@1, U$2.RTN_BATV_SW3@2, U$3.RTN_+3V3@1, U$3.RTN_+3V3@2, U$3.RTN_+3V3@3, U$3.RTN_+3V3@4, U$3.RTN_BATV@1, U$3.RTN_BATV@2, U$3.RTN_BATV@3, U$3.RTN_BATV@4, U1.FBLDO, U10.GND, U2.FBLDO, U3.FBLDO, U7.GND, U8.GND; no longer BATTERY.2, X1-BOT.GND@1, X1-BOT.GND@10, X1-BOT.GND@11, X1-BOT.GND@12, X1-BOT.GND@13, X1-BOT.GND@14, X1-BOT.GND@15, X1-BOT.GND@16, X1-BOT.GND@17, X1-BOT.GND@18, X1-BOT.GND@19, X1-BOT.GND@2, X1-BOT.GND@3, X1-BOT.GND@4, X1-BOT.GND@5, X1-BOT.GND@6, X1-BOT.GND@7, X1-BOT.GND@8, X1-BOT.GND@9, X1-TOP.GND@1, X1-TOP.GND@10, X1-TOP.GND@11, X1-TOP.GND@12, X1-TOP.GND@13, X1-TOP.GND@14, X1-TOP.GND@15, X1-TOP.GND@16, X1-TOP.GND@17, X1-TOP.GND@18, X1-TOP.GND@19, X1-TOP.GND@2, X1-TOP.GND@3, X1-TOP.GND@4, X1-TOP.GND@5, X1-TOP.GND@6, X1-TOP.GND@7, X1-TOP.GND@8, X1-TOP.GND@9
- net I2C_SCL: now also R8.2, SLAVE_SCL.1, U10.SCL; no longer X1-BOT.SCL, X1-TOP.SCL
- net I2C_SDA: now also R7.2, SLAVE_SDA.1, U10.SDA; no longer X1-BOT.SDA, X1-TOP.SDA
- net N$5: now also R11.2
- net N$6: now also R9.2
- net N$7: now also R14.2
- net N$8: now also R4.1, U8.ILIM; no longer BATTERY.1, SWITCH.1
Other:
- note added: "Overcurrent Protection"
- note added: "Voltage Regulator"
- note added: "Voltage Supervisor"
- moved on the sheet: C10, C9, L4, SOLAR_PANELS, U$1, U6

Commit message: Complteded routing
Parts:
- removed SLAVE_GND, SLAVE_SCL, SLAVE_SDA, SLAVE_VS: (no value), jumper:SJ
- added R15, R16, R17: 466k, adafruit:R-US_R0805
- added R18: 487, adafruit:R-US_R0805
- added R19: (no value), adafruit:R-US_R0805
- added U9: BQ24210DQCT, BQ24210:BQ24210DQCT
- BATTERY: value 332-02 -> (none); device con-garry:332-02 -> adafruit:PINHD-1X3
- R1, R2: value (none) -> 470k
Connections:
- removed net $N70: BATTERY-1.S, C8.2, SWITCH-1.S, U5.OUTA, U5.OUTB
- removed net I2C_SCL: R8.2, SLAVE_SCL.1, U10.SCL
- removed net I2C_SDA: R7.2, SLAVE_SDA.1, U10.SDA
- removed net N$18: SLAVE_GND.2, SLAVE_SCL.2, SLAVE_SDA.2, SLAVE_VS.2, U10.A0
- new net N$28: R15.2, U2.MPPC
- new net N$29: R16.2, U3.MPPC
- new net N$30: R17.2, U1.MPPC
- new net N$31: C8.2, U5.OUTA, U5.OUTB, U9.VBUS
- new net N$32: U9.~EN, U9.~PG
- new net N$33: R18.2, U9.ISET
- new net N$34: BATTERY.1, SWITCH-1.S, U9.BAT
- new net N$35: BATTERY.2, R19.2, U9.TS
- new net N$36: R19.1, U9.VTSB
- net !RST: now also U$3./RST
- net +3V3: no longer SLAVE_VS.1
- net BATV: now also SWITCH-2.S
- net GND: now also BATTERY.3, R15.1, R16.1, R17.1, R18.1, U10.EPAD, U9.EP, U9.VSS; no longer BATTERY-2.S, SLAVE_GND.1
- net GPIO0: now also U$3.GPIO0
- net GPIO1: now also U$3.GPIO1
- net SCL: now also R8.2, U$3.SCL, U10.A0, U10.SCL
- net SDA: now also R7.2, U$3.SDA, U10.SDA
Other:
- moved on the sheet: C10, C9, L4, SWITCH-1, SWITCH-2, U6

Commit message: many many things
Parts:
- removed R7, R8: 10k, adafruit:R-US_R0805
- removed U10: INA3221AIRGVT, INA3221:INA3221AIRGVT
Connections:
- removed net VIN1+: U10.IN+1
- removed net VIN1-: U10.IN-1
- removed net VIN2+: U10.IN+2
- removed net VIN2-: U10.IN-2
- removed net VIN3+: U10.IN+3
- removed net VIN3-: U10.IN-3
- net +3V3: no longer R7.1, R8.1, U10.VS
- net +3V3_SW1: now also U$3.+3V3_SW1@2
- net GND: now also U$3.GND, U$3.RTN_+3V3_SW1@1, U$3.RTN_+3V3_SW1@2, U$3.RTN_+3V3_SW2@1, U$3.RTN_+3V3_SW2@2, U$3.RTN_+3V3_SW3@1, U$3.RTN_+3V3_SW3@2, U$3.RTN_BATV_SW1@1, U$3.RTN_BATV_SW1@2, U$3.RTN_BATV_SW2@1, U$3.RTN_BATV_SW2@2, U$3.RTN_BATV_SW3@1, U$3.RTN_BATV_SW3@2; no longer U10.EPAD, U10.GND
- net SCL: no longer R8.2, U10.A0, U10.SCL
- net SDA: no longer R7.2, U10.SDA
Changed lines of the file:
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@@
 <classes>
 <class number="0" name="default" width="0" drill="0">
+<clearance class="0" value="0.205"/>
 </class>
 </classes>
@@
 <part name="SJ1" library="jumper" deviceset="SJ" device=""/>
 <part name="SJ2" library="jumper" deviceset="SJ" device=""/>
-<part name="U10" library="INA3221" deviceset="INA3221AIRGVT" device=""/>
-<part name="GND32" library="supply1" deviceset="GND" device=""/>
-<part name="R7" library="adafruit" deviceset="R-US_" device="R0805" value="10k"/>
-<part name="R8" library="adafruit" deviceset="R-US_" device="R0805" value="10k"/>
 <part name="C11" library="adafruit" deviceset="C-US" device="C0805" value="4.7uF"/>
 <part name="GND33" library="supply1" deviceset="GND" device=""/>
@@
 <instance part="SJ1" gate="1" x="480.06" y="363.22"/>
 <instance part="SJ2" gate="1" x="480.06" y="403.86"/>
-<instance part="U10" gate="A" x="149.86" y="294.64"/>
-<instance part="GND32" gate="1" x="124.46" y="281.94" rot="MR90"/>
-<instance part="R7" gate="G$1" x="185.42" y="256.54" rot="R90"/>
-<instance part="R8" gate="G$1" x="177.8" y="256.54" rot="R90"/>
 <instance part="C11" gate="G$1" x="266.7" y="414.02" rot="R180"/>
 <instance part="GND33" gate="1" x="266.7" y="421.64" rot="MR180"/>
@@
 <wire x1="474.98" y1="347.98" x2="485.14" y2="347.98" width="0.1524" layer="91"/>
 <wire x1="485.14" y1="347.98" x2="485.14" y2="353.06" width="0.1524" layer="91"/>
-</segment>
-<segment>
-<pinref part="U10" gate="A" pin="GND"/>
-<wire x1="129.54" y1="281.94" x2="127" y2="281.94" width="0.1524" layer="91"/>
-<pinref part="GND32" gate="1" pin="GND"/>
-<pinref part="U10" gate="A" pin="EPAD"/>
-<wire x1="129.54" y1="279.4" x2="129.54" y2="281.94" width="0.1524" layer="91"/>
-<junction x="129.54" y="281.94"/>
 </segment>
 <segment>
@@
 </segment>
 <segment>
-<wire x1="58.42" y1="96.52" x2="53.34" y2="96.52" width="0.1524" layer="91"/>
 <wire x1="53.34" y1="96.52" x2="53.34" y2="93.98" width="0.1524" layer="91"/>
 <wire x1="53.34" y1="93.98" x2="53.34" y2="86.36" width="0.1524" layer="91"/>
@@
 <wire x1="53.34" y1="43.18" x2="53.34" y2="33.02" width="0.1524" layer="91"/>
 <wire x1="53.34" y1="33.02" x2="53.34" y2="20.32" width="0.1524" layer="91"/>
+<pinref part="GND11" gate="1" pin="GND"/>
+<pinref part="U$3" gate="G$1" pin="GND"/>
 <wire x1="58.42" y1="33.02" x2="53.34" y2="33.02" width="0.1524" layer="91"/>
 <junction x="53.34" y="33.02"/>
+<pinref part="U$3" gate="G$1" pin="RTN_BATV_SW3@2"/>
+<wire x1="58.42" y1="43.18" x2="53.34" y2="43.18" width="0.1524" layer="91"/>
+<junction x="53.34" y="43.18"/>
+<pinref part="U$3" gate="G$1" pin="RTN_BATV_SW3@1"/>
 <wire x1="58.42" y1="45.72" x2="53.34" y2="45.72" width="0.1524" layer="91"/>
 <junction x="53.34" y="45.72"/>
-<wire x1="58.42" y1="43.18" x2="53.34" y2="43.18" width="0.1524" layer="91"/>
-<junction x="53.34" y="43.18"/>
+<pinref part="U$3" gate="G$1" pin="RTN_BATV_SW2@2"/>
+<wire x1="58.42" y1="53.34" x2="53.34" y2="53.34" width="0.1524" layer="91"/>
+<junction x="53.34" y="53.34"/>
+<pinref part="U$3" gate="G$1" pin="RTN_BATV_SW2@1"/>
 <wire x1="58.42" y1="55.88" x2="53.34" y2="55.88" width="0.1524" layer="91"/>
 <junction x="53.34" y="55.88"/>
-<wire x1="58.42" y1="53.34" x2="53.34" y2="53.34" width="0.1524" layer="91"/>
-<junction x="53.34" y="53.34"/>
+<pinref part="U$3" gate="G$1" pin="RTN_BATV_SW1@2"/>
+<wire x1="58.42" y1="63.5" x2="53.34" y2="63.5" width="0.1524" layer="91"/>
+<junction x="53.34" y="63.5"/>
+<pinref part="U$3" gate="G$1" pin="RTN_BATV_SW1@1"/>
 <wire x1="58.42" y1="66.04" x2="53.34" y2="66.04" width="0.1524" layer="91"/>
 <junction x="53.34" y="66.04"/>
-<wire x1="58.42" y1="63.5" x2="53.34" y2="63.5" width="0.1524" layer="91"/>
-<junction x="53.34" y="63.5"/>
+<pinref part="U$3" gate="G$1" pin="RTN_+3V3_SW3@2"/>
+<wire x1="58.42" y1="73.66" x2="53.34" y2="73.66" width="0.1524" layer="91"/>
+<junction x="53.34" y="73.66"/>
+<pinref part="U$3" gate="G$1" pin="RTN_+3V3_SW3@1"/>
 <wire x1="58.42" y1="76.2" x2="53.34" y2="76.2" width="0.1524" layer="91"/>
 <junction x="53.34" y="76.2"/>
-<wire x1="58.42" y1="73.66" x2="53.34" y2="73.66" width="0.1524" layer="91"/>
-<junction x="53.34" y="73.66"/>
+<pinref part="U$3" gate="G$1" pin="RTN_+3V3_SW2@2"/>
+<wire x1="58.42" y1="83.82" x2="53.34" y2="83.82" width="0.1524" layer="91"/>
+<junction x="53.34" y="83.82"/>
+<pinref part="U$3" gate="G$1" pin="RTN_+3V3_SW2@1"/>
 <wire x1="58.42" y1="86.36" x2="53.34" y2="86.36" width="0.1524" layer="91"/>
 <junction x="53.34" y="86.36"/>
-<wire x1="58.42" y1="83.82" x2="53.34" y2="83.82" width="0.1524" layer="91"/>
-<junction x="53.34" y="83.82"/>
+<pinref part="U$3" gate="G$1" pin="RTN_+3V3_SW1@2"/>
 <wire x1="58.42" y1="93.98" x2="53.34" y2="93.98" width="0.1524" layer="91"/>
 <junction x="53.34" y="93.98"/>
-<pinref part="GND11" gate="1" pin="GND"/>
+<pinref part="U$3" gate="G$1" pin="RTN_+3V3_SW1@1"/>
+<wire x1="58.42" y1="96.52" x2="53.34" y2="96.52" width="0.1524" layer="91"/>
 </segment>
 <segment>
@@
 </segment>
 <segment>
-<pinref part="U10" gate="A" pin="VS"/>
-<wire x1="114.3" y1="284.48" x2="129.54" y2="284.48" width="0.1524" layer="91"/>
-<label x="109.22" y="284.48" size="1.778" layer="95"/>
-</segment>
-<segment>
-<pinref part="R8" gate="G$1" pin="1"/>
-<wire x1="177.8" y1="251.46" x2="177.8" y2="243.84" width="0.1524" layer="91"/>
-<label x="177.8" y="241.3" size="1.778" layer="95" rot="R90"/>
-</segment>
-<segment>
-<pinref part="R7" gate="G$1" pin="1"/>
-<wire x1="185.42" y1="251.46" x2="185.42" y2="243.84" width="0.1524" layer="91"/>
-<label x="185.42" y="241.3" size="1.778" layer="95" rot="R90"/>
-</segment>
-<segment>
 <pinref part="U$2" gate="G$1" pin="+3V3@1"/>
 <wire x1="109.22" y1="193.04" x2="116.84" y2="193.04" width="0.1524" layer="91"/>
@@
 </segment>
 </net>
-<net name="VIN1-" class="0">
-<segment>
-<pinref part="U10" gate="A" pin="IN-1"/>
-<wire x1="129.54" y1="304.8" x2="124.46" y2="304.8" width="0.1524" layer="91"/>
-<label x="119.38" y="304.8" size="1.778" layer="95"/>
-</segment>
-</net>
-<net name="VIN1+" class="0">
-<segment>
-<pinref part="U10" gate="A" pin="IN+1"/>
-<wire x1="129.54" y1="302.26" x2="124.46" y2="302.26" width="0.1524" layer="91"/>
-<label x="119.38" y="302.26" size="1.778" layer="95"/>
-</segment>
-</net>
-<net name="VIN2-" class="0">
-<segment>
-<pinref part="U10" gate="A" pin="IN-2"/>
-<wire x1="129.54" y1="299.72" x2="124.46" y2="299.72" width="0.1524" layer="91"/>
-<label x="119.38" y="299.72" size="1.778" layer="95"/>
-</segment>
-</net>
-<net name="VIN2+" class="0">
-<segment>
-<pinref part="U10" gate="A" pin="IN+2"/>
-<wire x1="129.54" y1="297.18" x2="124.46" y2="297.18" width="0.1524" layer="91"/>
-<label x="119.38" y="297.18" size="1.778" layer="95"/>
-</segment>
-</net>
-<net name="VIN3-" class="0">
-<segment>
-<pinref part="U10" gate="A" pin="IN-3"/>
-<wire x1="129.54" y1="294.64" x2="124.46" y2="294.64" width="0.1524" layer="91"/>
-<label x="119.38" y="294.64" size="1.778" layer="95"/>
-</segment>
-</net>
-<net name="VIN3+" class="0">
-<segment>
-<pinref part="U10" gate="A" pin="IN+3"/>
-<wire x1="129.54" y1="292.1" x2="124.46" y2="292.1" width="0.1524" layer="91"/>
-<label x="119.38" y="292.1" size="1.778" layer="95"/>
-</segment>
-</net>
 <net name="N$19" class="0">
 <segment>
@@
 <label x="43.18" y="30.48" size="1.778" layer="95"/>
 </segment>
-<segment>
-<pinref part="R8" gate="G$1" pin="2"/>
-<pinref part="U10" gate="A" pin="SCL"/>
-<wire x1="170.18" y1="284.48" x2="177.8" y2="284.48" width="0.1524" layer="91"/>
-<wire x1="177.8" y1="284.48" x2="177.8" y2="261.62" width="0.1524" layer="91"/>
-<label x="177.8" y="284.48" size="1.778" layer="95"/>
-<pinref part="U10" gate="A" pin="A0"/>
-<wire x1="170.18" y1="287.02" x2="170.18" y2="284.48" width="0.1524" layer="91"/>
-<junction x="170.18" y="284.48"/>
-</segment>
 </net>
 <net name="SDA" class="0">
@@
 <wire x1="58.42" y1="27.94" x2="48.26" y2="27.94" width="0.1524" layer="91"/>
 <label x="43.18" y="27.94" size="1.778" layer="95"/>
-</segment>
-<segment>
-<pinref part="U10" gate="A" pin="SDA"/>
-<label x="175.26" y="304.8" size="1.778" layer="95"/>
-<pinref part="R7" gate="G$1" pin="2"/>
-<wire x1="170.18" y1="304.8" x2="185.42" y2="304.8" width="0.1524" layer="91"/>
-<wire x1="185.42" y1="304.8" x2="185.42" y2="261.62" width="0.1524" layer="91"/>
 </segment>
 </net>
@@
 <wire x1="58.42" y1="101.6" x2="50.8" y2="101.6" width="0.1524" layer="91"/>
 <wire x1="50.8" y1="101.6" x2="50.8" y2="99.06" width="0.1524" layer="91"/>
-<wire x1="50.8" y1="99.06" x2="58.42" y2="99.06" width="0.1524" layer="91"/>
 <wire x1="50.8" y1="101.6" x2="48.26" y2="101.6" width="0.1524" layer="91"/>
 <junction x="50.8" y="101.6"/>
 <label x="35.56" y="101.6" size="1.778" layer="95"/>
-</segment>
-</net>
+<pinref part="U$3" gate="G$1" pin="+3V3_SW1@2"/>
+<wire x1="50.8" y1="99.06" x2="58.42" y2="99.06" width="0.1524" layer="91"/>
+</segment>
+</net>
