File: Schematics/EPS/Flight Model/PQ60 EPS FV3.sch (EAGLE design)
At the start: 54 parts, among them U1 LTC3105EDDPBF, U2 LTC3105EDDPBF, U3 LTC3105EDDPBF, U4 LTC4413EDDPBF, U5 LTC4413EDDPBF, U6 TPS63001DRCR, U7 TPS2552DBVT, U8 TPS2552DBVT, U9 BQ24210DQCT

Commit message: Upddates
Parts:
- removed BATTERY: (no value), adafruit:PINHD-1X3
- removed SJ1, SJ2: (no value), jumper:SJ
- removed SOLAR_PANELS: (no value), adafruit:PINHD-1X12-CB
- removed SWITCH: 332-02, con-garry:332-02
- added R20, R21, R22, R23, R7, R8: 35.7k, adafruit:R-US_R0805
- added U$10, U$4, U$5, U$6, U$7, U$8, U$9: JST-SH-02, JST SH 02:JST-SH-02
- added U$11: JST-SH-03, JST SH 03:JST-SH-03
- added U10: PCA9534PW, PCA9534PW:PCA9534PW
- added U11, U12, U13: TPS2552DBVT, TPS2552:TPS2552DBVT
- R18: value 487 -> 787
- R19: value (none) -> 21.5k
Connections:
- new net N$38: R20.1, U12.ILIM
- new net N$39: R21.2, U12.~FAULT
- new net N$40: R22.1, U13.ILIM
- new net N$41: R23.2, U13.~FAULT
- new net SW1_EN: U10.IO0, U11.EN
- new net SW2_EN: U10.IO1, U12.EN
- new net SW3_EN: U10.IO2, U13.EN
- net +3V3: now also U10.VDD
- net +3V3_SW1: now also U11.OUT
- net +3V3_SW2: now also U12.OUT
- net +3V3_SW3: now also U13.OUT
- net BATTERY: now also U7.EN
- net BATV: now also U$10.P$2; no longer SWITCH-2.S
- net GND: now also R20.2, R22.2, R7.2, U$11.P$3, U$4.P$2, U$5.P$2, U$6.P$2, U$7.P$2, U$8.P$2, U$9.P$2, U10.VSS, U11.GND, U12.GND, U13.GND; no longer BATTERY.3, SJ1.1, SJ2.1, SOLAR_PANELS.10, SOLAR_PANELS.12, SOLAR_PANELS.2, SOLAR_PANELS.4, SOLAR_PANELS.6, SOLAR_PANELS.8
- net N$16: now also R7.1, U11.ILIM; no longer SJ1.2, U8.EN
- net N$17: now also R8.2, U11.~FAULT; no longer SJ2.2, U7.EN
- net N$34: now also U$10.P$1, U$11.P$1; no longer BATTERY.1, SWITCH-1.S
- net N$35: now also U$11.P$2; no longer BATTERY.2
- net PANEL1+2: now also U$4.P$1, U$5.P$1; no longer SOLAR_PANELS.1, SOLAR_PANELS.3
- net PANEL3+4: now also U$6.P$1, U$7.P$1; no longer SOLAR_PANELS.5, SOLAR_PANELS.7
- net PANEL5+6: now also U$8.P$1, U$9.P$1; no longer SOLAR_PANELS.11, SOLAR_PANELS.9
- net SCL: now also U10.SCL
- net SDA: now also U10.SDA
- net UNPROTECTED3V3: now also R21.1, R23.1, R8.1, U11.IN, U12.IN, U13.IN, U8.EN
Other:
- moved on the sheet: R5, U$3
