File: Schematics/EPS/Flight Model/PQ60 EPS FV2.brd (EAGLE design)
At the start: 42 x 42 mm, 54 parts, among them U1 LTC3105EDDPBF, U2 LTC3105EDDPBF, U3 LTC3105EDDPBF, U4 LTC4413EDDPBF, U5 LTC4413EDDPBF, U6 TPS63001DRCR, U7 TPS2552DBVT, U8 TPS2552DBVT, U9 BQ24210DQCT

Commit message: many changes
Parts:
- renumbered BATTERY to BATTERYPLUG
Connections:
- net BATTERY: now also U7.1; no longer R5.1, U7.6
- net BATV: now also R5.1, U7.6; no longer U7.1
Routing:
- net BATV: track 72.1 -> 84.5 mm
- net BATTERY: track 18.8 -> 15.6 mm
Changed lines of the file:
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@@
 <?xml version="1.0" encoding="utf-8"?>
 <!DOCTYPE eagle SYSTEM "eagle.dtd">
-<eagle version="7.3.0">
+<eagle version="7.4.0">
 <drawing>
 <settings>
@@
 <layer number="35" name="tGlue" color="7" fill="4" visible="no" active="yes"/>
 <layer number="36" name="bGlue" color="7" fill="5" visible="no" active="yes"/>
-<layer number="37" name="tTest" color="7" fill="1" visible="yes" active="yes"/>
+<layer number="37" name="tTest" color="7" fill="1" visible="no" active="yes"/>
 <layer number="38" name="bTest" color="7" fill="1" visible="yes" active="yes"/>
 <layer number="39" name="tKeepout" color="4" fill="11" visible="yes" active="yes"/>
@@
 <layer number="49" name="Reference" color="7" fill="1" visible="no" active="yes"/>
 <layer number="50" name="dxf" color="7" fill="1" visible="no" active="no"/>
-<layer number="51" name="tDocu" color="7" fill="1" visible="no" active="yes"/>
+<layer number="51" name="tDocu" color="7" fill="1" visible="yes" active="yes"/>
 <layer number="52" name="bDocu" color="7" fill="1" visible="no" active="yes"/>
 <layer number="53" name="tGND_GNDA" color="7" fill="1" visible="no" active="no"/>
@@
 <text x="26.4" y="38.7" size="1" layer="22" font="vector" rot="MR0">5</text>
 <text x="31.7" y="38.7" size="1" layer="22" font="vector" rot="MR0">6</text>
+<wire x1="5.7" y1="21.5" x2="9.7" y2="21.5" width="0.15" layer="51"/>
+<wire x1="9.7" y1="21.5" x2="9.7" y2="19.5" width="0.15" layer="51"/>
+<wire x1="9.7" y1="19.5" x2="5.7" y2="19.5" width="0.15" layer="51"/>
+<wire x1="5.7" y1="19.5" x2="5.7" y2="21.5" width="0.15" layer="51"/>
+<wire x1="9.7" y1="21.5" x2="13.7" y2="21.5" width="0.15" layer="51"/>
+<wire x1="13.7" y1="21.5" x2="13.7" y2="19.5" width="0.15" layer="51"/>
+<wire x1="13.7" y1="19.5" x2="9.7" y2="19.5" width="0.15" layer="51"/>
+<wire x1="7.7" y1="19.3" x2="11.7" y2="19.3" width="0.15" layer="51"/>
+<wire x1="11.7" y1="19.3" x2="11.7" y2="17.3" width="0.15" layer="51"/>
+<wire x1="11.7" y1="17.3" x2="7.7" y2="17.3" width="0.15" layer="51"/>
+<wire x1="7.7" y1="17.3" x2="7.7" y2="19.3" width="0.15" layer="51"/>
+<wire x1="5.7" y1="26.7" x2="7.7" y2="26.7" width="0.15" layer="51"/>
+<wire x1="7.7" y1="26.7" x2="7.7" y2="22.7" width="0.15" layer="51"/>
+<wire x1="7.7" y1="22.7" x2="5.7" y2="22.7" width="0.15" layer="51"/>
+<wire x1="5.7" y1="22.7" x2="5.7" y2="26.7" width="0.15" layer="51"/>
+<wire x1="8.2" y1="26.2" x2="11.2" y2="26.2" width="0.15" layer="51"/>
+<wire x1="11.2" y1="26.2" x2="11.2" y2="23.2" width="0.15" layer="51"/>
+<wire x1="11.2" y1="23.2" x2="8.2" y2="23.2" width="0.15" layer="51"/>
+<wire x1="8.2" y1="23.2" x2="8.2" y2="26.2" width="0.15" layer="51"/>
+<wire x1="11.7" y1="26.7" x2="13.7" y2="26.7" width="0.15" layer="51"/>
+<wire x1="13.7" y1="26.7" x2="13.7" y2="22.7" width="0.15" layer="51"/>
+<wire x1="13.7" y1="22.7" x2="11.7" y2="22.7" width="0.15" layer="51"/>
+<wire x1="11.7" y1="22.7" x2="11.7" y2="26.7" width="0.15" layer="51"/>
+<wire x1="7.7" y1="29.4" x2="11.7" y2="29.4" width="0.15" layer="51"/>
+<wire x1="11.7" y1="29.4" x2="11.7" y2="27.4" width="0.15" layer="51"/>
+<wire x1="11.7" y1="27.4" x2="7.7" y2="27.4" width="0.15" layer="51"/>
+<wire x1="7.7" y1="27.4" x2="7.7" y2="29.4" width="0.15" layer="51"/>
 </plain>
 <attributes>
@@
 </autorouter>
 <elements>
-<element name="BATTERY" library="adafruit" package="1X03" value="" x="40.2" y="10" smashed="yes" rot="R90">
+<element name="BATTERYPLUG" library="adafruit" package="1X03" value="" x="40.2" y="10" smashed="yes" rot="R90">
 <attribute name="NAME" x="40.7712" y="14.3138" size="1.27" layer="25" ratio="10" rot="R90"/>
 <attribute name="VALUE" x="43.375" y="6.19" size="1.27" layer="27" rot="R90"/>
@@
 <contactref element="R1" pad="2"/>
 <contactref element="R2" pad="2"/>
-<contactref element="U7" pad="1"/>
 <contactref element="SWITCH" pad="2"/>
 <wire x1="23.1" y1="4.775" x2="23.7" y2="4.775" width="0.254" layer="1"/>
@@
 <wire x1="24.3" y1="4.15" x2="23.7" y2="4.15" width="0.254" layer="16"/>
 <wire x1="23.7" y1="4.15" x2="23.1" y2="4.15" width="0.254" layer="16"/>
-<wire x1="24.0602" y1="15.4046" x2="24.0602" y2="14.1398" width="0.254" layer="1"/>
 <wire x1="28.775" y1="12.475" x2="31.5" y2="9.75" width="0.254" layer="1"/>
 <wire x1="31.5" y1="9.75" x2="31.5" y2="1.4" width="0.254" layer="1"/>
@@
 <wire x1="25.35" y1="0.55" x2="24.9" y2="1" width="0.254" layer="1"/>
 <wire x1="24.9" y1="1" x2="24.9" y2="6.5" width="0.254" layer="1"/>
+<contactref element="U7" pad="6"/>
+<contactref element="R5" pad="1"/>
+<wire x1="24.0602" y1="14.1398" x2="20.5" y2="14.1398" width="0.15" layer="1"/>
+<wire x1="20.5" y1="14.1398" x2="20.5" y2="18.2" width="0.15" layer="1"/>
+<wire x1="20.5" y1="18.2" x2="24.0602" y2="18.2" width="0.15" layer="1"/>
+<wire x1="24.0602" y1="18.2" x2="24.0602" y2="17.9954" width="0.15" layer="1"/>
+<wire x1="24.0602" y1="17.9954" x2="24" y2="17.9954" width="0.15" layer="1"/>
+<wire x1="24" y1="17.9954" x2="24" y2="20.2" width="0.15" layer="1"/>
 </signal>
 <signal name="+3V3">
@@
 <contactref element="U9" pad="3"/>
 <contactref element="R18" pad="1"/>
-<contactref element="BATTERY" pad="3"/>
+<contactref element="BATTERYPLUG" pad="3"/>
 <wire x1="16.5" y1="9.85" x2="15.9" y2="9.85" width="0.254" layer="16"/>
 <wire x1="18.9" y1="9.85" x2="18.3" y2="9.85" width="0.254" layer="16"/>
@@
 </signal>
 <signal name="BATTERY">
-<contactref element="U7" pad="6"/>
-<contactref element="R5" pad="1"/>
 <contactref element="U6" pad="7"/>
 <contactref element="U6" pad="6"/>
@@
 <contactref element="U6" pad="5"/>
 <contactref element="C9" pad="2"/>
-<wire x1="24.0602" y1="17.9954" x2="24.1" y2="17.9954" width="0.254" layer="1"/>
-<wire x1="24.0602" y1="17.9954" x2="24" y2="17.9954" width="0.254" layer="1"/>
-<wire x1="24" y1="17.9954" x2="24" y2="20.2" width="0.254" layer="1"/>
 <wire x1="28.5906" y1="26.8732" x2="28.108" y2="26.8732" width="0.254" layer="1"/>
 <wire x1="28.108" y1="26.8732" x2="27.6" y2="26.8732" width="0.254" layer="1"/>
@@
 <wire x1="26.5" y1="21.5" x2="24.4" y2="21.5" width="0.254" layer="1"/>
 <wire x1="24.4" y1="21.5" x2="24" y2="21.1" width="0.254" layer="1"/>
-<wire x1="24" y1="21.1" x2="24" y2="20.2" width="0.254" layer="1"/>
 <wire x1="28.9" y1="21.4" x2="27.9" y2="21.4" width="0.254" layer="1"/>
 <wire x1="28.5906" y1="23.9268" x2="28.9268" y2="23.9268" width="0.254" layer="1"/>
@@
 <wire x1="27" y1="21" x2="27.5" y2="21" width="0.254" layer="1"/>
 <wire x1="27.5" y1="21" x2="27.9" y2="21.4" width="0.254" layer="1"/>
+<contactref element="U7" pad="1"/>
+<wire x1="24.0602" y1="15.4046" x2="24" y2="21.1" width="0" layer="19" extent="1-1"/>
 </signal>
 <signal name="UNPROTECTED3V3">
@@
 <contactref element="U9" pad="10"/>
 <contactref element="SWITCH" pad="1"/>
-<contactref element="BATTERY" pad="1"/>
+<contactref element="BATTERYPLUG" pad="1"/>
 <wire x1="36" y1="5.5" x2="34" y2="5.5" width="0.254" layer="1"/>
 <wire x1="34" y1="5.5" x2="33.6" y2="5.9" width="0.254" layer="1"/>
@@
 </signal>
 <signal name="N$35">
-<contactref element="BATTERY" pad="2"/>
+<contactref element="BATTERYPLUG" pad="2"/>
 <contactref element="U9" pad="5"/>
 <contactref element="R19" pad="2"/>
