File: Schematics/EPS/Flight Model/PQ60 EPS FV3.brd (EAGLE design)
At the start: 42 x 42 mm, 67 parts, among them U1 LTC3105EDDPBF, U10 PCA9534PW, U11 TPS2552DBVT, U12 TPS2552DBVT, U13 TPS2552DBVT, U2 LTC3105EDDPBF, U3 LTC3105EDDPBF, U4 LTC4413EDDPBF, U5 LTC4413EDDPBF, U6 TPS63001DRCR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

Commit message: many changes
Connections:
- net BATTERY: now also U$10.P2
- net BATV: no longer U$10.P2
Routing:
- net BATTERY: track 22.3 -> 45.0 mm, vias 0 -> 4
- net GND: track 154.4 -> 149.8 mm, vias 16 -> 15
- net BATV: track 116.6 -> 114.8 mm
Changed lines of the file:
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@@
 <wire x1="28.8046" y1="24.8954" x2="28.8" y2="24.9" width="0.254" layer="1"/>
 <via x="28.8" y="24.9" extent="1-16" drill="0.3"/>
-<contactref element="U$10" pad="P2"/>
-<wire x1="36.85" y1="33.45" x2="36.85" y2="31.65" width="0.3" layer="1"/>
 <via x="36.85" y="31.65" extent="1-16" drill="0.3"/>
 <wire x1="36.85" y1="31.65" x2="36.85" y2="29.65" width="0.3" layer="16"/>
@@
 <wire x1="31.6738" y1="32.9202" x2="33.1216" y2="32.9202" width="0.254" layer="1"/>
 <wire x1="34.0106" y1="33.8092" x2="34.6202" y2="33.8092" width="0.254" layer="1"/>
-<wire x1="29.438" y1="26.976" x2="29.438" y2="26.65" width="0.254" layer="16"/>
 <wire x1="5.4" y1="31.95" x2="2.6" y2="31.95" width="0.4064" layer="1"/>
 <wire x1="11.4" y1="33.8" x2="12.7762" y2="33.8" width="0.4064" layer="1"/>
@@
 <wire x1="8.4" y1="27" x2="11.25" y2="27" width="0.4064" layer="1"/>
 <wire x1="11.25" y1="27" x2="11.4" y2="27.15" width="0.4064" layer="1"/>
-<wire x1="29.438" y1="26.976" x2="29.2602" y2="26.976" width="0.1524" layer="16"/>
-<wire x1="29.2602" y1="26.976" x2="28.2448" y2="25.9606" width="0.1524" layer="16"/>
-<wire x1="28.2448" y1="25.9606" x2="27.305" y2="25.9606" width="0.1524" layer="16"/>
-<wire x1="27.305" y1="25.9606" x2="26.797" y2="25.4526" width="0.1524" layer="16"/>
-<wire x1="26.797" y1="25.4526" x2="25.8064" y2="25.4526" width="0.1524" layer="16"/>
-<via x="25.8064" y="25.4526" extent="1-16" drill="0.3"/>
 <wire x1="25.8064" y1="25.4526" x2="25.8064" y2="27.1436" width="0.1524" layer="1"/>
 <wire x1="25.8064" y1="27.1436" x2="25.8" y2="27.15" width="0.1524" layer="1"/>
@@
 <wire x1="39.2" y1="11.4" x2="38.6" y2="12" width="0.1524" layer="1"/>
 <wire x1="38.6" y1="14.3" x2="38.7" y2="14.4" width="0.1524" layer="1"/>
+<wire x1="14.478" y1="25.3002" x2="14.5752" y2="27.15" width="0" layer="19" extent="1-1"/>
 <wire x1="39.5954" y1="14.4" x2="39.7" y2="14.3" width="0" layer="19" extent="1-16"/>
 </signal>
@@
 <wire x1="30.5" y1="22.3" x2="31.3852" y2="22.3" width="0.254" layer="1"/>
 <wire x1="31.3852" y1="22.3" x2="31.3954" y2="22.3102" width="0.254" layer="1"/>
+<contactref element="U$10" pad="P2"/>
+<wire x1="36.85" y1="33.45" x2="36.85" y2="32.7" width="0.254" layer="1"/>
+<via x="36.85" y="32.7" extent="1-16" drill="0.3"/>
+<wire x1="36.85" y1="32.7" x2="37.65" y2="33.5" width="0.254" layer="16"/>
+<wire x1="37.65" y1="33.5" x2="40.3" y2="33.5" width="0.254" layer="16"/>
+<via x="40.3" y="33.5" extent="1-16" drill="0.3"/>
+<wire x1="40.3" y1="33.5" x2="39.95" y2="33.5" width="0.254" layer="1"/>
+<wire x1="39.95" y1="33.5" x2="39.4" y2="32.95" width="0.254" layer="1"/>
+<wire x1="39.4" y1="32.95" x2="39.4" y2="26.75" width="0.254" layer="1"/>
+<wire x1="39.4" y1="26.75" x2="36.85" y2="24.2" width="0.254" layer="1"/>
+<via x="36.85" y="24.2" extent="1-16" drill="0.3"/>
+<wire x1="36.85" y1="24.2" x2="34.5" y2="24.2" width="0.254" layer="16"/>
+<wire x1="34.5" y1="24.2" x2="31.7" y2="21.45" width="0.254" layer="16"/>
+<via x="31.7" y="21.45" extent="1-16" drill="0.3"/>
+<wire x1="31.7" y1="21.45" x2="31.7" y2="22.0056" width="0.254" layer="1"/>
+<wire x1="31.7" y1="22.0056" x2="31.3954" y2="22.3102" width="0.254" layer="1"/>
 </signal>
 <signal name="UNPROTECTED3V3">
