File: Schematics/EPS/Flight Model/PQ60 EPS FV4.brd (EAGLE design)
At the start: 42 x 42 mm, 101 parts, among them U1 LTC3105EDDPBF, U10 PCA9534PW, U11 DRV, U12 DRV, U13 LTC4413EDDPBF, U14 DRV, U15 DRV, U16 LTC4413EDDPBF, U17 DRV, U18 DRV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

Commit message: m
Parts:
- C17, C19, C20, C24, C25, C27, C31, C33: value 4.7uF -> 0.1uF
- C18, C23, C26, C28, C29, C30, C32, C34: value .1uF -> 0.1uF
Other:
- board text added: "EPS FV4"
- board text added: "S^3"
- board text added: "simplespacesystems.com"
Changed lines of the file:
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@@
 <wire x1="32.5" y1="39.275" x2="32.775" y2="39" width="0.15" layer="22" curve="90"/>
 <circle x="28.85" y="11.35" radius="0.05" width="0.4064" layer="21"/>
+<text x="28.3" y="0.55" size="1.27" layer="21">EPS FV4</text>
+<text x="32.95" y="2.2" size="1.27" layer="21">S^3</text>
+<text x="41" y="21" size="1.27" layer="22" rot="MR270" align="center">simplespacesystems.com</text>
 </plain>
 <attributes>
@@
 </element>
 <element name="R3" library="adafruit" package="R0805" value="100k" x="37.025" y="27.85" smashed="yes" rot="MR270"/>
-<element name="C17" library="adafruit" package="C0805" value="4.7uF" x="38.025" y="28.875" smashed="yes"/>
-<element name="C18" library="adafruit" package="C0805" value=".1uF" x="38.025" y="26.85" smashed="yes" rot="R180"/>
+<element name="C17" library="adafruit" package="C0805" value="0.1uF" x="38.025" y="28.875" smashed="yes"/>
+<element name="C18" library="adafruit" package="C0805" value="0.1uF" x="38.025" y="26.85" smashed="yes" rot="R180"/>
 <element name="R4" library="adafruit" package="R0805" value="35.7k" x="39.075" y="27.85" smashed="yes" rot="MR270"/>
 <element name="U8" library="TPS2552" package="DRV" value="DRV" x="37.375" y="13.3" rot="R90"/>
 <element name="R5" library="adafruit" package="R0805" value="100k" x="34.625" y="17.45" smashed="yes" rot="MR180"/>
-<element name="C25" library="adafruit" package="C0805" value="4.7uF" x="33.65" y="18.425" smashed="yes" rot="R90"/>
-<element name="C26" library="adafruit" package="C0805" value=".1uF" x="35.725" y="18.45" smashed="yes" rot="R270"/>
+<element name="C25" library="adafruit" package="C0805" value="0.1uF" x="33.65" y="18.425" smashed="yes" rot="R90"/>
+<element name="C26" library="adafruit" package="C0805" value="0.1uF" x="35.725" y="18.45" smashed="yes" rot="R270"/>
 <element name="R6" library="adafruit" package="R0805" value="35.7k" x="34.65" y="19.525" smashed="yes" rot="MR0"/>
 <element name="U17" library="TPS2552" package="DRV" value="DRV" x="23.3" y="12.675" rot="R90"/>
-<element name="C27" library="adafruit" package="C0805" value="4.7uF" x="25.9" y="17.425" smashed="yes"/>
-<element name="C28" library="adafruit" package="C0805" value=".1uF" x="25.9" y="19.525" smashed="yes" rot="R180"/>
+<element name="C27" library="adafruit" package="C0805" value="0.1uF" x="25.9" y="17.425" smashed="yes"/>
+<element name="C28" library="adafruit" package="C0805" value="0.1uF" x="25.9" y="19.525" smashed="yes" rot="R180"/>
 <element name="R31" library="adafruit" package="R0805" value="35.7k" x="27.05" y="18.5" smashed="yes" rot="MR90"/>
 <element name="R30" library="adafruit" package="R0805" value="100k" x="24.9" y="18.5" smashed="yes" rot="MR270"/>
 <element name="U14" library="TPS2552" package="DRV" value="DRV" x="34.1" y="8.45"/>
-<element name="C19" library="adafruit" package="C0805" value="4.7uF" x="38.15" y="8.975" smashed="yes"/>
-<element name="C29" library="adafruit" package="C0805" value=".1uF" x="38.15" y="11.05" smashed="yes"/>
+<element name="C19" library="adafruit" package="C0805" value="0.1uF" x="38.15" y="8.975" smashed="yes"/>
+<element name="C29" library="adafruit" package="C0805" value="0.1uF" x="38.15" y="11.05" smashed="yes"/>
 <element name="R24" library="adafruit" package="R0805" value="35.7k" x="39.275" y="10.05" smashed="yes" rot="MR90"/>
 <element name="R25" library="adafruit" package="R0805" value="100k" x="37.125" y="10.075" smashed="yes" rot="MR270"/>
 <element name="U11" library="TPS2552" package="DRV" value="DRV" x="20.2" y="12.675" rot="R90"/>
-<element name="C24" library="adafruit" package="C0805" value="4.7uF" x="21.7" y="17.425" smashed="yes"/>
-<element name="C30" library="adafruit" package="C0805" value=".1uF" x="21.7" y="19.525" smashed="yes"/>
+<element name="C24" library="adafruit" package="C0805" value="0.1uF" x="21.7" y="17.425" smashed="yes"/>
+<element name="C30" library="adafruit" package="C0805" value="0.1uF" x="21.7" y="19.525" smashed="yes"/>
 <element name="R7" library="adafruit" package="R0805" value="35.7k" x="22.525" y="18.5" smashed="yes" rot="MR90"/>
 <element name="R8" library="adafruit" package="R0805" value="100k" x="20.425" y="18.5" smashed="yes" rot="MR270"/>
 <element name="U18" library="TPS2552" package="DRV" value="DRV" x="29.725" y="13" smashed="yes"/>
-<element name="C31" library="adafruit" package="C0805" value="4.7uF" x="33.875" y="12.025" smashed="yes"/>
-<element name="C32" library="adafruit" package="C0805" value=".1uF" x="33.875" y="14.1" smashed="yes" rot="R180"/>
+<element name="C31" library="adafruit" package="C0805" value="0.1uF" x="33.875" y="12.025" smashed="yes"/>
+<element name="C32" library="adafruit" package="C0805" value="0.1uF" x="33.875" y="14.1" smashed="yes" rot="R180"/>
 <element name="R32" library="adafruit" package="R0805" value="35.7k" x="35" y="13.1" smashed="yes" rot="MR90"/>
 <element name="R33" library="adafruit" package="R0805" value="100k" x="32.85" y="13.1" smashed="yes" rot="MR270"/>
 <element name="U12" library="TPS2552" package="DRV" value="DRV" x="17.1" y="12.675" rot="R90"/>
-<element name="C20" library="adafruit" package="C0805" value="4.7uF" x="17.525" y="17.425" smashed="yes"/>
-<element name="C23" library="adafruit" package="C0805" value=".1uF" x="17.525" y="19.525" smashed="yes"/>
+<element name="C20" library="adafruit" package="C0805" value="0.1uF" x="17.525" y="17.425" smashed="yes"/>
+<element name="C23" library="adafruit" package="C0805" value="0.1uF" x="17.525" y="19.525" smashed="yes"/>
 <element name="R20" library="adafruit" package="R0805" value="35.7k" x="17.95" y="18.5" smashed="yes" rot="MR90"/>
 <element name="R21" library="adafruit" package="R0805" value="100k" x="15.775" y="18.5" smashed="yes" rot="MR270"/>
 <element name="U15" library="TPS2552" package="DRV" value="DRV" x="26.45" y="12.75" rot="R90"/>
-<element name="C33" library="adafruit" package="C0805" value="4.7uF" x="30.075" y="17.425" smashed="yes"/>
-<element name="C34" library="adafruit" package="C0805" value=".1uF" x="30.075" y="19.525" smashed="yes"/>
+<element name="C33" library="adafruit" package="C0805" value="0.1uF" x="30.075" y="17.425" smashed="yes"/>
+<element name="C34" library="adafruit" package="C0805" value="0.1uF" x="30.075" y="19.525" smashed="yes"/>
 <element name="R26" library="adafruit" package="R0805" value="35.7k" x="31.35" y="18.5" smashed="yes" rot="MR90"/>
 <element name="R27" library="adafruit" package="R0805" value="100k" x="29.225" y="18.5" smashed="yes" rot="MR270"/>
@@
 <wire x1="30.167" y1="23.842" x2="29.4768" y2="23.842" width="0.254" layer="1"/>
 <via x="29.475" y="27.45" extent="1-16" drill="0.3"/>
-<via x="31.675" y="0.775" extent="1-16" drill="0.3"/>
+<via x="27.375" y="0.625" extent="1-16" drill="0.3"/>
 <via x="2.45" y="8.075" extent="1-16" drill="0.3"/>
 <via x="39" y="26.85" extent="1-16" drill="0.3"/>
