File: Schematics/Radio/Flight Model/PQ60 Radio FV1/PQ60 Radio FV1.brd (EAGLE design)
At the start: 42 x 42 mm, 2 parts

Commit message: Upddates
Parts:
- added C1: 47uF, adafruit:C0805
- added C2: 100nF, adafruit:C0805
- added CX2156NL: CX2156NL, CX2156NL:CX2156NL
- added U$1: RF4463F30, Radio EV1:RF4463F30
- added U$4: MICRO-SMA, Micro-sma:MICRO-SMA
Connections:
- removed net RTN_+3V3_SW1: U$3.P$3, U$3.P$4
- removed net RTN_+3V3_SW2: U$3.P$7, U$3.P$8
- removed net RTN_+3V3_SW3: U$3.P$11, U$3.P$12
- removed net RTN_BATV_SW1: U$3.P$15, U$3.P$16
- removed net RTN_BATV_SW2: U$3.P$19, U$3.P$20
- removed net RTN_BATV_SW3: U$3.P$23, U$3.P$24
- new net N$1: CX2156NL.1, U$1.P$16
- new net N$2: CX2156NL.6, U$4.SIGNAL
- new net N$3: CX2156NL.4, U$4.GND@1, U$4.GND@2, U$4.GND@3
- net BATV: now also C1.1, C2.1, U$1.P$1
- net GND: now also C1.2, C2.2, CX2156NL.3, U$1.P$15, U$1.P$2, U$1.P$8, U$3.P$11, U$3.P$12, U$3.P$15, U$3.P$16, U$3.P$19, U$3.P$20, U$3.P$23, U$3.P$24, U$3.P$28, U$3.P$3, U$3.P$4, U$3.P$7, U$3.P$8
- net GPIO10: now also U$1.P$7
- net GPIO2: now also U$1.P$6
- net GPIO8: now also U$1.P$12
- net GPIO9: now also U$1.P$5
- net MISO: now also U$1.P$11
- net MOSI: now also U$1.P$10
- net SCK: now also U$1.P$9
Routing:
- net GPIO8: track 0.00 -> 52.5 mm, vias 0 -> 1
- net SCK: track 0.00 -> 50.1 mm, vias 0 -> 2
- net MOSI: track 0.00 -> 46.8 mm, vias 0 -> 2
- net MISO: track 0.00 -> 44.3 mm, vias 0 -> 2
- net GPIO9: track 0.00 -> 43.1 mm, vias 0 -> 2
- net +3V3: track 38.2 -> 8.25 mm, vias 4 -> 1
- net GPIO2: track 0.00 -> 28.8 mm, vias 0 -> 1
- net GND: track 75.6 -> 98.7 mm, vias 6 -> 10
- net GPIO10: track 0.00 -> 20.8 mm, vias 0 -> 1
- net N$3: track 0.00 -> 9.80 mm
- net GPIO5: track 0.00 -> 6.37 mm, vias 0 -> 1
- net N$2: track 0.00 -> 5.74 mm
- net GPIO7: track 0.00 -> 5.13 mm, vias 0 -> 1
- net GPIO3: track 0.00 -> 5.13 mm, vias 0 -> 1
- net GPIO11: track 0.00 -> 5.13 mm, vias 0 -> 1
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- added copper zone on layer 1, net GND
- added copper zone on layer 16, net GND
Other:
- board text added: "Radio FV1"
- board text added: "Radio Goes Here"
- board text added: "kartikye.com"
- board text removed: "+"
- board text removed: "-"
