File: Schematics/FlatSat/flatsat.brd (EAGLE design)
At the start: 100 x 100 mm, 9 parts

Commit message: many changes
Routing:
- net BATV_SW2: track 246.9 -> 245.8 mm
- net +3V3: track 252.9 -> 253.8 mm
- net MOSI: track 245.0 -> 245.8 mm
- net +3V3_SW2: track 221.3 -> 221.9 mm
- net GPIO11: track 221.9 -> 222.4 mm
Other:
- outline, holes or cut-outs redrawn
