File: Schematics/Radio/Flight Model/PQ60 Radio FV1.sch (EAGLE design)
At the start: 7 parts

Commit message: Upddates
Connections:
- net +3V3: now also U$3.+3V3@1, U$3.+3V3@2, U$3.+3V3@3, U$3.+3V3@4
- net +3V3_SW1: now also U$3.+3V3_SW1@1
- net +3V3_SW2: now also U$3.+3V3_SW2@1, U$3.+3V3_SW2@2
- net +3V3_SW3: now also U$3.+3V3_SW3@1, U$3.+3V3_SW3@2
- net BATV: now also U$3.BATV@1, U$3.BATV@2, U$3.BATV@3, U$3.BATV@4
- net BATV_SW1: now also U$3.BATV_SW1@1, U$3.BATV_SW1@2
- net BATV_SW2: now also U$3.BATV_SW2@1, U$3.BATV_SW2@2
- net BATV_SW3: now also U$3.BATV_SW3@1, U$3.BATV_SW3@2
- net GPIO10: now also U$1.NSEL; no longer U$1.GPIO1
- net GPIO11: no longer U$1.NIRQ
- net GPIO12: no longer U$1.SDN
- net GPIO2: now also U$1.NIRQ
- net GPIO8: now also U$1.GPIO1
- net GPIO9: now also U$1.SDN; no longer U$1.NSEL
