File: Schematics/Radio/Flight Model/PQ60 Radio FV1.brd (EAGLE design)
At the start: 42 x 42 mm, 7 parts

Commit message: Upddates
Connections:
- net GPIO10: now also U$1.P$7; no longer U$1.P$12
- net GPIO11: no longer U$1.P$6
- net GPIO12: no longer U$1.P$5
- net GPIO2: now also U$1.P$6
- net GPIO8: now also U$1.P$12
- net GPIO9: now also U$1.P$5; no longer U$1.P$7
Routing:
- net GPIO8: track 4.97 -> 52.5 mm
- net GPIO12: track 42.2 -> 3.53 mm, vias 2 -> 1
- net GPIO10: track 51.7 -> 20.8 mm, vias 2 -> 1
- net GPIO2: track 3.53 -> 28.8 mm
- net GPIO11: track 27.4 -> 5.13 mm
- net GPIO9: track 25.0 -> 43.1 mm, vias 1 -> 2
- net +3V3_SW1: track 3.28 -> 2.68 mm
Other:
- board text added: "Radio FV1"
- board text added: "Radio Goes Here"
- board text added: "kartikye.com"

Commit message: many changes
Routing:
- net GPIO9: track 43.1 -> 44.7 mm
Changed lines of the file:
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@@
 <via x="31" y="12.2" extent="1-16" drill="0.3"/>
 <wire x1="31" y1="12.2" x2="31.2" y2="12.2" width="0.254" layer="16"/>
-<wire x1="31.2" y1="12.2" x2="31.7" y2="11.7" width="0.254" layer="16"/>
-<wire x1="31.7" y1="11.7" x2="31.7" y2="2.2" width="0.254" layer="16"/>
-<wire x1="31.7" y1="2.2" x2="30.7" y2="1.2" width="0.254" layer="16"/>
 <wire x1="30.7" y1="1.2" x2="19" y2="1.2" width="0.254" layer="16"/>
 <wire x1="19" y1="1.2" x2="18.3" y2="1.9" width="0.254" layer="16"/>
+<wire x1="31.2" y1="12.2" x2="33.7" y2="9.7" width="0.254" layer="16"/>
+<wire x1="33.7" y1="9.7" x2="33.7" y2="4.2" width="0.254" layer="16"/>
+<wire x1="33.7" y1="4.2" x2="30.7" y2="1.2" width="0.254" layer="16"/>
 </signal>
 <signal name="GPIO10">

Commit message: m
Other:
- board text added: "+"
- board text added: "-"
- board text added: "0.1uF"
- board text added: "47uF"
- board text added: "S^3"
- board text added: "simplesapcesystems.com"
- board text removed: "kartikye.com"
Changed lines of the file:
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@@
 <wire x1="3" y1="0" x2="39" y2="0" width="0" layer="20"/>
 <wire x1="39" y1="0" x2="42" y2="3" width="0" layer="20" curve="90"/>
-<text x="15.4" y="18.6" size="2.54" layer="29">kartikye.com</text>
-<text x="6.1" y="39.7" size="1.27" layer="29">kartikye.com</text>
+<text x="21" y="16.5" size="1.778" layer="22" rot="MR0" align="center">simplesapcesystems.com</text>
+<text x="6.1" y="39.7" size="1.27" layer="29">S^3</text>
 <text x="6.1" y="38.1" size="1.27" layer="29">Radio FV1</text>
-<text x="36.2" y="0.3" size="1.27" layer="22" rot="MR0">Radio FV1</text>
-<text x="21" y="27" size="2.1844" layer="21" align="center">Radio Goes Here</text>
+<text x="21" y="27.5" size="2.54" layer="22" rot="MR0" align="center">Radio FV1</text>
+<text x="21" y="24.1" size="2.1844" layer="21" align="center">Radio Goes Here</text>
+<text x="0.8" y="7" size="1.778" layer="21">+</text>
+<text x="0.8" y="8.7" size="1.778" layer="21">-</text>
+<text x="1.6" y="5.9" size="0.8128" layer="21">47uF</text>
+<text x="5.4" y="5.9" size="0.8128" layer="21">0.1uF</text>
+<text x="21" y="21" size="5.08" layer="22" rot="MR0" align="center">S^3</text>
 </plain>
 <attributes>
