File: Schematics/CB/Flight Model/PQ60 CB FV2.brd (EAGLE design)
At the start: 42 x 42 mm, 26 parts, among them U1 ATMEGA328P-AU, U2 LSM9DS0, U3 LTC2990IMSPBF

Commit message: many changes
Parts:
- removed JP1: (no value), pinhead:1X02
- removed U$1: 10uF, AVE-4653:AVE-4653
- added C9: 10 uF Pol, adafruit:C0805
- added U$10: 6.8MM-BATTERY, 6.8mm-battery:6.8MM-BATTERY
- added U$7: JST-SH-02, JST SH 02:JST-SH-02
- added U$8: DS1388, DS1388:DS1388
- added U$9: AB25, AB25:ABS25
- moved C7 30.4 mm to (7.65, 37.9), turned to 0 degrees
- moved R5 29.7 mm to (18.6, 31.0), turned to 0 degrees
- moved SJ2 29.1 mm to (13.4, 30.5), flipped to the top, turned to 0 degrees
- moved SJ1 28.2 mm to (12.0, 28.3), flipped to the top
- moved R4 26.2 mm to (22.9, 31.0), turned to 0 degrees
- moved C5 24.3 mm to (10.7, 36.9), turned to 270 degrees
- moved U2 24.1 mm to (8.12, 32.2)
- moved U3 23.8 mm to (17.5, 26.8), turned to 270 degrees
- moved C6 23.0 mm to (7.65, 35.9)
- moved C2 22.1 mm to (1.13, 9.65), turned to 270 degrees
- moved C4 21.5 mm to (32.2, 2.25)
- moved C1 20.2 mm to (34.6, 5.69), turned to 270 degrees
- moved C3 18.6 mm to (1.13, 9.65), flipped to the bottom, turned to 270 degrees
- moved R3 16.9 mm to (7.00, 8.80), flipped to the bottom, turned to 90 degrees
- moved R2 13.0 mm to (8.00, 11.8), flipped to the bottom, turned to 0 degrees
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Connections:
- new net N$14: U$10.P$1
- new net N$18: U$8.P$1, U$9.P$1
- new net N$19: U$8.P$2, U$9.P$4
- new net N$20: U$10.P$3, U$8.P$3
- net !RST: now also U$8.P$7
- net +3V3: now also C9.2, U$8.P$8; no longer U$1.+
- net GND: now also C9.1, U$10.P$2, U$8.P$4; no longer U$1.-
- net N$10: now also U$7.P2; no longer JP1.2
- net N$11: now also U$7.P1; no longer JP1.1
- net SCL: now also U$8.P$6
- net SDA: now also U$8.P$5
Routing:
- net +3V3: track 132.1 -> 234.6 mm, vias 7 -> 12
- net BATV: track 28.1 -> 102.6 mm
- net GND: track 101.8 -> 152.9 mm, vias 10 -> 20
- net CHASSIS_GND: track 118.4 -> 79.8 mm, vias 4 -> 3
- net !RST: track 60.5 -> 94.4 mm, vias 1 -> 5
- net SCK: track 84.3 -> 115.3 mm
- net GPIO10: track 60.7 -> 39.0 mm, vias 3 -> 2
- net GPIO6: track 51.5 -> 32.8 mm, vias 2 -> 3
- net GPIO5: track 48.4 -> 30.4 mm, vias 2 -> 1
- net N$8: track 21.1 -> 5.27 mm, vias 1 -> 2
- net GPIO7: track 46.6 -> 31.8 mm
- net GPIO9: track 50.7 -> 38.2 mm, vias 1 -> 2
- net GPIO11: track 31.9 -> 43.6 mm, vias 2 -> 3
- net GPIO12: track 32.7 -> 43.7 mm, vias 2 -> 3
- net GPIO8: track 51.3 -> 40.8 mm, vias 3 -> 2
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- added copper zone on layer 1, net GND
- added copper zone on layer 16, net GND
Other:
- board text added: "+"
- board text added: "-"
- board text removed: "SASSat EPS FV2"

Commit message: m
Parts:
- moved U$4 0.26 mm to (1.50, 13.7), flipped to the bottom
Routing:
- net GND: track 152.9 -> 154.5 mm, vias 20 -> 22
- net MOSI: track 100.9 -> 102.0 mm, vias 4 -> 6
- net N$2: track 8.51 -> 8.79 mm, vias 1 -> 2
- net N$3: track 9.88 -> 9.97 mm, vias 2 -> 1
Other:
- board text added: "Control Board FV2"
- board text added: "Simple Space Systems"
- board text added: "simplespacesystems.com"
