File: Schematics/CB/Flight Model/PQ60 CB FV2.sch (EAGLE design)
At the start: 26 parts, among them U1 ATMEGA328P-AU, U2 LSM9DS0, U3 LTC2990IMSPBF

Commit message: many changes
Parts:
- removed JP1: (no value), pinhead:PINHD-1X2
- removed U$1: 10uF, AVE-4653:AVE-4653
- added C9: 10 uF Pol, adafruit:C-USC0805
- added U$10: 6.8MM-BATTERY, 6.8mm-battery:6.8MM-BATTERY
- added U$7: JST-SH-02, JST SH 02:JST-SH-02
- added U$8: DS1388, DS1388:DS1388
- added U$9: AB25, AB25:AB25
Connections:
- new net N$14: U$10.VCC@1
- new net N$18: U$8.X1, U$9.X1
- new net N$19: U$8.X2, U$9.X2
- new net N$20: U$10.VCC@2, U$8.V_BACKUP
- net !RST: now also U$8.!RST
- net +3V3: now also C9.2, U$8.VCC; no longer U$1.+
- net GND: now also C9.1, U$10.GND, U$8.GND; no longer U$1.-
- net N$10: now also U$7.P$2; no longer JP1.2
- net N$11: now also U$7.P$1; no longer JP1.1
- net SCL: now also U$8.SCL
- net SDA: now also U$8.SDA
Other:
- note removed: "10uF"
Changed lines of the file:
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@@
 <?xml version="1.0" encoding="utf-8"?>
 <!DOCTYPE eagle SYSTEM "eagle.dtd">
-<eagle version="7.3.0">
+<eagle version="7.4.0">
 <drawing>
 <settings>
@@
 <part name="C7" library="rcl" deviceset="C-EU" device="C0805" value="100nF"/>
 <part name="GND4" library="supply1" deviceset="GND" device=""/>
-<part name="U$1" library="AVE-4653" deviceset="AVE-4653" device="" value="10uF"/>
 <part name="R2" library="adafruit" deviceset="R-US_" device="M0805" value="10k"/>
 <part name="R3" library="adafruit" deviceset="R-US_" device="M0805" value="10k"/>
@@
 <part name="C8" library="rcl" deviceset="C-EU" device="C0805" value="0.1uF"/>
 <part name="GND14" library="supply1" deviceset="GND" device=""/>
-<part name="JP1" library="pinhead" deviceset="PINHD-1X2" device=""/>
 <part name="U$5" library="1210-047J" deviceset="1210-047J" device=""/>
 <part name="U$6" library="mircosd" deviceset="MICROSD" device=""/>
 <part name="GND15" library="supply1" deviceset="GND" device=""/>
+<part name="U$7" library="JST SH 02" deviceset="JST-SH-02" device=""/>
+<part name="U$8" library="DS1388" deviceset="DS1388" device=""/>
+<part name="GND16" library="supply1" deviceset="GND" device=""/>
+<part name="U$9" library="AB25" deviceset="AB25" device=""/>
+<part name="U$10" library="6.8mm-battery" deviceset="6.8MM-BATTERY" device=""/>
+<part name="C9" library="adafruit" deviceset="C-US" device="C0805" value="10 uF Pol"/>
 </parts>
 <sheets>
 <sheet>
 <plain>
-<text x="76.2" y="398.78" size="1.778" layer="91">10uF</text>
 <text x="118.11" y="281.305" size="1.27" layer="95">RX</text>
 <text x="118.11" y="278.765" size="1.27" layer="95">TX</text>
@@
 <instance part="C6" gate="G$1" x="68.58" y="363.22" rot="R180"/>
 <instance part="C7" gate="G$1" x="58.42" y="383.54" rot="R180"/>
-<instance part="GND4" gate="1" x="53.34" y="408.94" rot="MR90"/>
-<instance part="U$1" gate="G$1" x="73.66" y="378.46" rot="R90"/>
+<instance part="GND4" gate="1" x="55.88" y="391.16" rot="MR90"/>
 <instance part="R2" gate="G$1" x="81.28" y="220.98"/>
 <instance part="R3" gate="G$1" x="81.28" y="210.82"/>
@@
 <instance part="C8" gate="G$1" x="162.56" y="299.72" rot="R180"/>
 <instance part="GND14" gate="1" x="162.56" y="309.88" rot="R180"/>
-<instance part="JP1" gate="G$1" x="152.4" y="271.78" rot="R180"/>
 <instance part="U$5" gate="A" x="45.72" y="297.18"/>
 <instance part="U$6" gate="G$1" x="167.64" y="223.52"/>
 <instance part="GND15" gate="1" x="134.62" y="226.06" rot="R270"/>
+<instance part="U$7" gate="G$1" x="157.48" y="271.78" rot="R180"/>
+<instance part="U$8" gate="G$1" x="218.44" y="193.04"/>
+<instance part="GND16" gate="1" x="187.96" y="185.42" rot="R270"/>
+<instance part="U$9" gate="G$1" x="177.8" y="203.2" rot="R180"/>
+<instance part="U$10" gate="G$1" x="177.8" y="175.26" rot="R90"/>
+<instance part="C9" gate="G$1" x="68.58" y="386.08"/>
 </instances>
 <busses>
@@
 </segment>
 <segment>
-<pinref part="U$1" gate="G$1" pin="-"/>
 <pinref part="GND4" gate="1" pin="GND"/>
-<wire x1="68.58" y1="406.4" x2="68.58" y2="408.94" width="0.1524" layer="91"/>
-<wire x1="68.58" y1="408.94" x2="58.42" y2="408.94" width="0.1524" layer="91"/>
 <pinref part="C7" gate="G$1" pin="2"/>
-<wire x1="58.42" y1="408.94" x2="55.88" y2="408.94" width="0.1524" layer="91"/>
-<wire x1="58.42" y1="388.62" x2="58.42" y2="408.94" width="0.1524" layer="91"/>
-<junction x="58.42" y="408.94"/>
+<wire x1="68.58" y1="391.16" x2="58.42" y2="391.16" width="0.1524" layer="91"/>
+<wire x1="58.42" y1="388.62" x2="58.42" y2="391.16" width="0.1524" layer="91"/>
+<junction x="58.42" y="391.16"/>
+<pinref part="C9" gate="G$1" pin="1"/>
+<wire x1="68.58" y1="388.62" x2="68.58" y2="391.16" width="0.1524" layer="91"/>
 </segment>
 <segment>
@@
 <wire x1="157.48" y1="226.06" x2="137.16" y2="226.06" width="0.1524" layer="91"/>
 <pinref part="GND15" gate="1" pin="GND"/>
+</segment>
+<segment>
+<pinref part="U$8" gate="G$1" pin="GND"/>
+<wire x1="200.66" y1="185.42" x2="190.5" y2="185.42" width="0.1524" layer="91"/>
+<pinref part="GND16" gate="1" pin="GND"/>
+<pinref part="U$10" gate="G$1" pin="GND"/>
+<wire x1="185.42" y1="175.26" x2="190.5" y2="175.26" width="0.1524" layer="91"/>
+<wire x1="190.5" y1="175.26" x2="190.5" y2="185.42" width="0.1524" layer="91"/>
+<junction x="190.5" y="185.42"/>
 </segment>
 </net>
@@
 <wire x1="58.42" y1="381" x2="58.42" y2="378.46" width="0.1524" layer="91"/>
 <junction x="58.42" y="378.46"/>
-<wire x1="68.58" y1="381" x2="68.58" y2="378.46" width="0.1524" layer="91"/>
+<wire x1="68.58" y1="388.62" x2="68.58" y2="381" width="0.1524" layer="91"/>
 <junction x="68.58" y="378.46"/>
 <pinref part="U2" gate="G$1" pin="VDD_IO"/>
+<wire x1="68.58" y1="381" x2="68.58" y2="378.46" width="0.1524" layer="91"/>
 <wire x1="68.58" y1="378.46" x2="68.58" y2="375.92" width="0.1524" layer="91"/>
 <wire x1="68.58" y1="375.92" x2="71.12" y2="375.92" width="0.1524" layer="91"/>
-<pinref part="U$1" gate="G$1" pin="+"/>
-<wire x1="68.58" y1="375.92" x2="45.72" y2="375.92" width="0.1524" layer="91"/>
+<wire x1="68.58" y1="375.92" x2="48.26" y2="375.92" width="0.1524" layer="91"/>
 <junction x="68.58" y="375.92"/>
-<wire x1="45.72" y1="375.92" x2="45.72" y2="411.48" width="0.1524" layer="91"/>
-<wire x1="45.72" y1="411.48" x2="104.14" y2="411.48" width="0.1524" layer="91"/>
+<wire x1="48.26" y1="375.92" x2="48.26" y2="393.7" width="0.1524" layer="91"/>
+<wire x1="48.26" y1="393.7" x2="104.14" y2="393.7" width="0.1524" layer="91"/>
 <pinref part="U2" gate="G$1" pin="CS(G)"/>
-<wire x1="104.14" y1="411.48" x2="104.14" y2="370.84" width="0.1524" layer="91"/>
+<wire x1="104.14" y1="393.7" x2="104.14" y2="370.84" width="0.1524" layer="91"/>
 <wire x1="104.14" y1="370.84" x2="104.14" y2="365.76" width="0.1524" layer="91"/>
 <wire x1="104.14" y1="365.76" x2="101.6" y2="365.76" width="0.1524" layer="91"/>
@@
 <wire x1="101.6" y1="370.84" x2="104.14" y2="370.84" width="0.1524" layer="91"/>
 <junction x="104.14" y="370.84"/>
+<pinref part="C9" gate="G$1" pin="2"/>
+<junction x="68.58" y="381"/>
 </segment>
 <segment>
@@
 <label x="142.24" y="231.14" size="1.27" layer="95" rot="R180" xref="yes"/>
 </segment>
+<segment>
+<pinref part="U$8" gate="G$1" pin="VCC"/>
+<wire x1="236.22" y1="200.66" x2="246.38" y2="200.66" width="0.1524" layer="91"/>
+<label x="246.38" y="200.66" size="1.27" layer="95" xref="yes"/>
+</segment>
 </net>
 <net name="!RST" class="0">
@@
 <wire x1="78.74" y1="327.66" x2="73.66" y2="327.66" width="0.1524" layer="91"/>
 <label x="73.66" y="327.66" size="1.27" layer="95" rot="R180" xref="yes"/>
+</segment>
+<segment>
+<pinref part="U$8" gate="G$1" pin="!RST"/>
+<wire x1="236.22" y1="195.58" x2="246.38" y2="195.58" width="0.1524" layer="91"/>
+<label x="246.38" y="195.58" size="1.27" layer="95" xref="yes"/>
 </segment>
 </net>
@@
 <label x="157.48" y="281.94" size="1.27" layer="95" rot="R180" xref="yes"/>
 </segment>
+<segment>
+<pinref part="U$8" gate="G$1" pin="SCL"/>
+<wire x1="236.22" y1="190.5" x2="246.38" y2="190.5" width="0.1524" layer="91"/>
+<label x="246.38" y="190.5" size="1.27" layer="95" xref="yes"/>
+</segment>
 </net>
 <net name="SDA" class="0">
@@
 <wire x1="200.66" y1="294.64" x2="208.28" y2="294.64" width="0.1524" layer="91"/>
 <label x="208.28" y="294.64" size="1.27" layer="95" xref="yes"/>
+</segment>
+<segment>
+<pinref part="U$8" gate="G$1" pin="SDA"/>
+<wire x1="236.22" y1="185.42" x2="246.38" y2="185.42" width="0.1524" layer="91"/>
+<label x="246.38" y="185.42" size="1.27" layer="95" xref="yes"/>
 </segment>
 </net>
@@
 </segment>
 </net>
-<net name="N$10" class="0">
-<segment>
-<pinref part="U3" gate="A" pin="V3"/>
-<pinref part="JP1" gate="G$1" pin="2"/>
-<wire x1="165.1" y1="271.78" x2="154.94" y2="271.78" width="0.1524" layer="91"/>
-</segment>
-</net>
-<net name="N$11" class="0">
-<segment>
-<pinref part="U3" gate="A" pin="V4"/>
-<pinref part="JP1" gate="G$1" pin="1"/>
-<wire x1="165.1" y1="269.24" x2="154.94" y2="269.24" width="0.1524" layer="91"/>
-</segment>
-</net>
 <net name="N$4" class="0">
 <segment>
@@
 </segment>
 </net>
+<net name="N$10" class="0">
+<segment>
+<pinref part="U3" gate="A" pin="V3"/>
+<pinref part="U$7" gate="G$1" pin="P$2"/>
+<wire x1="165.1" y1="271.78" x2="162.56" y2="271.78" width="0.1524" layer="91"/>
+</segment>
+</net>
+<net name="N$11" class="0">
+<segment>
+<pinref part="U3" gate="A" pin="V4"/>
+<pinref part="U$7" gate="G$1" pin="P$1"/>
+<wire x1="165.1" y1="269.24" x2="162.56" y2="269.24" width="0.1524" layer="91"/>
+</segment>
+</net>
+<net name="N$18" class="0">
+<segment>
+<pinref part="U$8" gate="G$1" pin="X1"/>
+<wire x1="200.66" y1="200.66" x2="190.5" y2="200.66" width="0.1524" layer="91"/>
+<pinref part="U$9" gate="G$1" pin="X1"/>
+</segment>
+</net>
+<net name="N$19" class="0">
+<segment>
+<pinref part="U$8" gate="G$1" pin="X2"/>
+<pinref part="U$9" gate="G$1" pin="X2"/>
+<wire x1="200.66" y1="195.58" x2="165.1" y2="195.58" width="0.1524" layer="91"/>
+<wire x1="165.1" y1="195.58" x2="165.1" y2="200.66" width="0.1524" layer="91"/>
+</segment>
+</net>
+<net name="N$20" class="0">
+<segment>
+<pinref part="U$8" gate="G$1" pin="V_BACKUP"/>
+<pinref part="U$10" gate="G$1" pin="VCC@2"/>
+<wire x1="200.66" y1="190.5" x2="177.8" y2="190.5" width="0.1524" layer="91"/>
+</segment>
+</net>
+<net name="N$14" class="0">
+<segment>
+<pinref part="U$10" gate="G$1" pin="VCC@1"/>
+<wire x1="177.8" y1="160.02" x2="177.8" y2="152.4" width="0.1524" layer="91"/>
+</segment>
+</net>

Commit message: m
Changed lines of the file:
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@@
 <junction x="58.42" y="391.16"/>
 <pinref part="C9" gate="G$1" pin="1"/>
-<wire x1="68.58" y1="388.62" x2="68.58" y2="391.16" width="0.1524" layer="91"/>
+<wire x1="68.58" y1="391.16" x2="68.58" y2="388.62" width="0.1524" layer="91"/>
 </segment>
 <segment>
@@
 <wire x1="58.42" y1="381" x2="58.42" y2="378.46" width="0.1524" layer="91"/>
 <junction x="58.42" y="378.46"/>
-<wire x1="68.58" y1="388.62" x2="68.58" y2="381" width="0.1524" layer="91"/>
 <junction x="68.58" y="378.46"/>
 <pinref part="U2" gate="G$1" pin="VDD_IO"/>
@@
 <junction x="104.14" y="370.84"/>
 <pinref part="C9" gate="G$1" pin="2"/>
-<junction x="68.58" y="381"/>
 </segment>
 <segment>
