File: Schematics/Radio/Enginnering Model/Radio EV1.brd (EAGLE design)
At the start: 45 x 35 mm, 5 parts

Commit message: m
Connections:
- net N$1 renamed NSEL
- net N$10 renamed VCC
- net N$2 renamed SDN
- net N$3 renamed NIRQ
- net N$4 renamed SCLK
- net N$5 renamed SDI
- net N$6 renamed SDO
- net N$7 renamed GPIO1
Changed lines of the file:
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@@
 <?xml version="1.0" encoding="utf-8"?>
 <!DOCTYPE eagle SYSTEM "eagle.dtd">
-<eagle version="7.2.0">
+<eagle version="7.4.0">
 <drawing>
 <settings>
@@
 <wire x1="32.5" y1="3.57" x2="31.72" y2="2.79" width="0.254" layer="1"/>
 </signal>
-<signal name="N$2">
+<signal name="SDN">
 <contactref element="U$1" pad="P$5"/>
 <contactref element="U$2" pad="2"/>
@@
 <wire x1="14" y1="2.85" x2="13.94" y2="2.79" width="0.254" layer="1"/>
 </signal>
-<signal name="N$3">
+<signal name="NIRQ">
 <contactref element="U$1" pad="P$6"/>
 <contactref element="U$2" pad="3"/>
@@
 <wire x1="16.48" y1="11.98" x2="16.5" y2="12" width="0.254" layer="1"/>
 </signal>
-<signal name="N$1">
+<signal name="NSEL">
 <contactref element="U$1" pad="P$7"/>
 <contactref element="U$2" pad="4"/>
@@
 <wire x1="19" y1="2.81" x2="19.02" y2="2.79" width="0.254" layer="1"/>
 </signal>
-<signal name="N$4">
+<signal name="SCLK">
 <contactref element="U$1" pad="P$9"/>
 <contactref element="U$2" pad="5"/>
@@
 <wire x1="8.5" y1="28.25" x2="8.5" y2="32" width="0.254" layer="1"/>
 </signal>
-<signal name="N$5">
+<signal name="SDI">
 <contactref element="U$1" pad="P$10"/>
 <contactref element="U$2" pad="6"/>
@@
 <wire x1="12.5" y1="28.25" x2="12.5" y2="32" width="0.254" layer="1"/>
 </signal>
-<signal name="N$6">
+<signal name="SDO">
 <contactref element="U$1" pad="P$11"/>
 <contactref element="U$2" pad="7"/>
@@
 <wire x1="16.5" y1="28.25" x2="16.5" y2="32" width="0.254" layer="1"/>
 </signal>
-<signal name="N$7">
+<signal name="GPIO1">
 <contactref element="U$1" pad="P$12"/>
 <contactref element="U$2" pad="8"/>
@@
 <wire x1="40.76" y1="27.74" x2="36.5" y2="32" width="0.254" layer="1"/>
 </signal>
-<signal name="N$10">
+<signal name="VCC">
 <contactref element="C2" pad="1"/>
 <contactref element="U$2" pad="1"/>
