File: Schematics/Radio/Enginnering Model/Radio EV1.sch (EAGLE design)
At the start: 5 parts

Commit message: m
Connections:
- net N$1 renamed NSEL
- net N$10 renamed VCC
- net N$2 renamed SDN
- net N$3 renamed NIRQ
- net N$4 renamed SCLK
- net N$5 renamed SDI
- net N$6 renamed SDO
- net N$7 renamed GPIO1
Changed lines of the file:
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@@
 <?xml version="1.0" encoding="utf-8"?>
 <!DOCTYPE eagle SYSTEM "eagle.dtd">
-<eagle version="7.2.0">
+<eagle version="7.4.0">
 <drawing>
 <settings>
@@
 </segment>
 </net>
-<net name="N$2" class="0">
+<net name="SDN" class="0">
 <segment>
 <pinref part="U$1" gate="G$1" pin="SDN"/>
@@
 </segment>
 </net>
-<net name="N$3" class="0">
+<net name="NIRQ" class="0">
 <segment>
 <pinref part="U$1" gate="G$1" pin="NIRQ"/>
@@
 </segment>
 </net>
-<net name="N$1" class="0">
+<net name="NSEL" class="0">
 <segment>
 <pinref part="U$1" gate="G$1" pin="NSEL"/>
@@
 </segment>
 </net>
-<net name="N$4" class="0">
+<net name="SCLK" class="0">
 <segment>
 <pinref part="U$1" gate="G$1" pin="SCLK"/>
@@
 </segment>
 </net>
-<net name="N$5" class="0">
+<net name="SDI" class="0">
 <segment>
 <pinref part="U$1" gate="G$1" pin="SDI"/>
@@
 </segment>
 </net>
-<net name="N$6" class="0">
+<net name="SDO" class="0">
 <segment>
 <pinref part="U$1" gate="G$1" pin="SDO"/>
@@
 </segment>
 </net>
-<net name="N$7" class="0">
+<net name="GPIO1" class="0">
 <segment>
 <pinref part="U$1" gate="G$1" pin="GPIO1"/>
@@
 </segment>
 </net>
-<net name="N$10" class="0">
+<net name="VCC" class="0">
 <segment>
 <pinref part="C2" gate="G$1" pin="1"/>
